Commit message: Rename laser_frame link to laser for consistency in lidar.xacro

File: urdf/lidar.xacro (robot description, xacro)
@@ -3,8 +3,8 @@
     <joint name="laser_joint" type="fixed">
         <parent link="chassis"/>
-        <child link="laser_frame"/>
+        <child link="laser"/>
         <origin xyz="0.122 0 0.212" rpy="0 0 0"/>
     </joint>
-    <link name="laser_frame">
+    <link name="laser">
         <visual>
             <geometry>

Commit message: Rename child link and associated link name to laser_frame for consistency in lidar.xacro

File: urdf/lidar.xacro (robot description, xacro)
@@ -3,8 +3,8 @@
     <joint name="laser_joint" type="fixed">
         <parent link="chassis"/>
-        <child link="laser"/>
+        <child link="laser_frame"/>
         <origin xyz="0.122 0 0.212" rpy="0 0 0"/>
     </joint>
-    <link name="laser">
+    <link name="laser_frame">
         <visual>
             <geometry>

Commit message: Fix parent link in laser_joint to base_link and update origin position in lidar.xacro

File: urdf/lidar.xacro (robot description, xacro)
@@ -2,7 +2,7 @@
 <robot xmlns:xacro="http://www.ros.org/wiki/xacro" >
     <joint name="laser_joint" type="fixed">
-        <parent link="chassis"/>
+        <parent link="base_link"/>
         <child link="laser_frame"/>
-        <origin xyz="0.122 0 0.212" rpy="0 0 0"/>
+        <origin xyz="0.0 0.0 0.02" rpy="0 0 0"/>
     </joint>
     <link name="laser_frame">
